File: caneval.kicad_pcb (KiCad board)
At the start: 2 copper layers, 49.5 x 19 mm, 15 parts, among them J1 CAN, J2 INPUT, T1 760390013, U1 ISO1044BD, U2 SN6505ADBV, U3 TPS76350

Commit message: add enable pin connection
Connections:
- U2 pad 5: unconnected-(U2-EN-Pad5) -> /VIN
Changed lines of the file:
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@@
 		(capping no)
 		(filling no)
-		(zone_defaults)
 		(pcbplotparams
 			(layerselection 0x00000000_00000000_55555555_5755f5ff)
@@
 			(layers "F.Cu" "F.Mask" "F.Paste")
 			(roundrect_rratio 0.25)
-			(net "unconnected-(U2-EN-Pad5)")
+			(net "/VIN")
 			(pinfunction "EN_5")
 			(pintype "input")
@@
 	)
 	(segment
+		(start 113.6375 97.462345)
+		(end 115.215155 99.04)
+		(width 0.5)
+		(layer "F.Cu")
+		(net "Net-(U2-D1)")
+	)
+	(segment
+		(start 115.215155 99.04)
+		(end 118.93 99.04)
+		(width 0.5)
+		(layer "F.Cu")
+		(net "Net-(U2-D1)")
+	)
+	(segment
 		(start 120.595 102.635)
 		(end 117.436393 102.635)
@@
 	)
 	(segment
-		(start 130.34 93.96)
-		(end 130.42 94.04)
-		(width 0.5)
-		(layer "F.Cu")
-		(net "Net-(D1-A)")
-	)
-	(segment
-		(start 128.07 93.96)
-		(end 130.34 93.96)
-		(width 0.5)
-		(layer "F.Cu")
-		(net "Net-(D1-A)")
-	)
-	(segment
-		(start 129.42 99.04)
-		(end 130.42 100.04)
-		(width 0.3)
-		(layer "F.Cu")
-		(net "Net-(D2-A)")
-	)
-	(segment
-		(start 128.07 99.04)
-		(end 129.42 99.04)
-		(width 0.3)
-		(layer "F.Cu")
-		(net "Net-(D2-A)")
-	)
-	(segment
-		(start 113.6375 97.462345)
-		(end 115.215155 99.04)
-		(width 0.5)
-		(layer "F.Cu")
-		(net "Net-(U2-D1)")
-	)
-	(segment
-		(start 115.215155 99.04)
-		(end 118.93 99.04)
-		(width 0.5)
-		(layer "F.Cu")
-		(net "Net-(U2-D1)")
-	)
-	(segment
 		(start 142.890001 100.130001)
 		(end 144.57 101.81)
@@
 		(net "/CAN_P")
 	)
+	(segment
+		(start 130.34 93.96)
+		(end 130.42 94.04)
+		(width 0.5)
+		(layer "F.Cu")
+		(net "Net-(D1-A)")
+	)
+	(segment
+		(start 128.07 93.96)
+		(end 130.34 93.96)
+		(width 0.5)
+		(layer "F.Cu")
+		(net "Net-(D1-A)")
+	)
+	(segment
+		(start 129.42 99.04)
+		(end 130.42 100.04)
+		(width 0.3)
+		(layer "F.Cu")
+		(net "Net-(D2-A)")
+	)
+	(segment
+		(start 128.07 99.04)
+		(end 129.42 99.04)
+		(width 0.3)
+		(layer "F.Cu")
+		(net "Net-(D2-A)")
+	)
 	(zone
