File: caneval.kicad_sch (KiCad schematic)
At the start: 15 parts, among them J1 CAN, J2 INPUT, T1 760390013, U1 ISO1044BD, U2 SN6505ADBV, U3 TPS76350

Commit message: add enable pin connection
Connections:
- net VIN: now also U2.5 (EN)
Changed lines of the file:
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@@
+	)
+	(junction
+		(at 39.37 31.75)
+		(diameter 0)
+		(color 0 0 0 0)
 	)
 	(junction
@@
 	(wire
 		(pts
+			(xy 39.37 41.91) (xy 39.37 31.75)
+		)
+		(stroke
+			(width 0)
+			(type default)
+		)
+	)
+	(wire
+		(pts
 			(xy 140.97 38.1) (xy 133.35 38.1)
 		)
@@
 	(wire
 		(pts
+			(xy 41.91 41.91) (xy 39.37 41.91)
+		)
+		(stroke
+			(width 0)
+			(type default)
+		)
+	)
+	(wire
+		(pts
 			(xy 110.49 40.64) (xy 110.49 48.26)
 		)
@@
 	(wire
 		(pts
-			(xy 35.56 31.75) (xy 71.12 31.75)
-		)
-		(stroke
+			(xy 39.37 31.75) (xy 71.12 31.75)
+		)
+		(stroke
+			(width 0)
+			(type default)
+		)
+	)
+	(wire
+		(pts
+			(xy 35.56 31.75) (xy 39.37 31.75)
+		)
+		(stroke
